File: PCB_desing/Hardwareproject.kicad_pcb (KiCad board)
At the start: 2 copper layers, 9 parts, among them J1 Barrel_Jack, Q1 IRF540N, T1 Transformer_1P_1S

Commit message: All PCB is done, average switch network is created and transfer function tested.
Parts:
- added C3: 18.8nF, Capacitor_THT:C_Disc_D3.4mm_W2.1mm_P2.50mm, F.Cu at (56.1, 125.0)
- added C4: 470nF, Capacitor_THT:C_Disc_D3.4mm_W2.1mm_P2.50mm, F.Cu at (68.3, 111.5)
- added C5: 100nF, Capacitor_THT:C_Disc_D3.4mm_W2.1mm_P2.50mm, F.Cu at (97.5, 113.1)
- added C6: 10nF, Capacitor_THT:C_Disc_D3.4mm_W2.1mm_P2.50mm, F.Cu at (68.3, 115.8)
- added J2: Conn_01x01, Connector:Banana_Jack_1Pin, F.Cu at (160.7, 65.1)
- added J3: Conn_01x01, Connector:Banana_Jack_1Pin, F.Cu at (161.1, 86.5)
- added J4: Barrel_Jack, Connector_BarrelJack:BarrelJack_CUI_PJ-063AH_Horizontal, F.Cu at (43.8, 81.3)
- added R3: 1000, Resistor_THT:R_Axial_DIN0204_L3.6mm_D1.6mm_P5.08mm_Horizontal, F.Cu at (56.1, 118.6)
- added R4: 270 ohm, Resistor_THT:R_Axial_DIN0204_L3.6mm_D1.6mm_P5.08mm_Horizontal, F.Cu at (74.4, 113.5)
- added R5: 30 ohm, Resistor_THT:R_Axial_DIN0204_L3.6mm_D1.6mm_P5.08mm_Horizontal, F.Cu at (89.1, 112.9)
- added R6: 200 ohm, Resistor_THT:R_Axial_DIN0204_L3.6mm_D1.6mm_P5.08mm_Horizontal, F.Cu at (83.3, 123.0)
- added U1: lt1246, Package_DIP:DIP-8_W7.62mm, F.Cu at (60.7, 109.0)
- C1: value 20u -> 200u; footprint Capacitor_SMD:CP_Elec_4x5.4 -> Capacitor_THT:CP_Radial_D7.5mm_P2.50mm
- C2: value 100u -> 330u; footprint Capacitor_THT:CP_Radial_D7.5mm_P2.50mm -> Capacitor_THT:CP_Radial_D12.5mm_P5.00mm
- D1: value D -> VT3080S; footprint Package_TO_SOT_THT:TO-220-2_Horizontal_TabDown -> Package_TO_SOT_THT:TO-220-2_Vertical
- D2: footprint Package_TO_SOT_THT:TO-220-2_Horizontal_TabDown -> Diode_THT:D_A-405_P7.62mm_Horizontal
- J1: footprint Connector_BarrelJack:BarrelJack_CUI_PJ-102AH_Horizontal -> Connector_BarrelJack:BarrelJack_CUI_PJ-063AH_Horizontal
- R1: value 1k -> 2k; footprint Resistor_SMD:R_0201_0603Metric -> Resistor_THT:R_Axial_DIN0204_L3.6mm_D1.6mm_P5.08mm_Horizontal
- R2: value 3 -> 1k; footprint Resistor_THT:R_Axial_DIN0204_L3.6mm_D1.6mm_P1.90mm_Vertical -> Resistor_THT:R_Axial_DIN0204_L3.6mm_D1.6mm_P5.08mm_Horizontal
- T1: value Transformer_1P_1S -> PA0184NL; footprint Transformer_THT:Transformer_CHK_EI30-2VA_1xSec -> Transformer_THT:Transformer_CHK_EI54-12VA_1xSec
- moved C1 122.7 mm to (62.8, 74.5), turned to 270 degrees
- moved J1 111.3 mm to (43.3, 111.0), turned to 270 degrees
- moved D2 103.9 mm to (61.3, 84.4), turned to 270 degrees
- moved R1 86.4 mm to (53.5, 82.2), turned to 90 degrees
- moved R2 82.5 mm to (92.9, 109.1)
- moved T1 54.7 mm to (80.4, 75.9)
- moved Q1 53.7 mm to (73.4, 99.8), turned to 90 degrees
- moved D1 44.9 mm to (122.8, 67.6)
- moved C2 40.3 mm to (141.7, 63.9), turned to 270 degrees
Connections:
- net Net-(J1-Pad2) renamed GND
- Q1 pad 1: (no net) -> Net-(Q1-Pad1)
- R2 pad 2: Net-(C2-Pad2) -> Net-(C4-Pad1)
- T1 pad 2: Net-(D2-Pad2) -> (no net)
- T1 pad 3: Net-(C2-Pad2) -> (no net)
- T1 pad 5: (no net) -> Net-(C2-Pad2)
- T1 pad 8: (no net) -> Net-(D2-Pad2)

Commit message: Updates
Parts:
- added HS1: Heatsink, Heatsink:Heatsink_Stonecold_HS-132_32x14mm_2xFixation1.5mm, F.Cu at (139.7, 47.0)
- added HS2: Heatsink, Heatsink:Heatsink_Stonecold_HS-132_32x14mm_2xFixation1.5mm, F.Cu at (73.7, 106.7)
- C3, C4, C5, C6: footprint Capacitor_THT:C_Disc_D3.4mm_W2.1mm_P2.50mm -> Capacitor_Tantalum_SMD:CP_EIA-3216-10_Kemet-I
- moved J1 46.4 mm to (40.6, 64.8)
- moved C4 32.1 mm to (100.2, 114.3), turned to 180 degrees
- moved R2 29.0 mm to (121.9, 107.7), turned to 180 degrees
- moved R5 28.6 mm to (117.7, 112.4), turned to 180 degrees
- moved C6 28.5 mm to (96.6, 118.5), turned to 180 degrees
- moved D1 28.3 mm to (142.2, 47.0), turned to 180 degrees
- moved C5 28.0 mm to (125.5, 112.1), turned to 180 degrees
- moved R6 25.1 mm to (107.8, 118.0), turned to 270 degrees
- moved R4 19.9 mm to (94.2, 114.3), turned to 180 degrees
- moved J4 15.5 mm to (40.6, 96.5)
- moved C2 8.72 mm to (143.5, 72.4)
- moved R1 8.53 mm to (53.5, 73.7), turned to 270 degrees
- moved R3 4.33 mm to (55.9, 114.3), turned to 270 degrees
- moved Q1 3.06 mm to (73.7, 102.9), turned to 270 degrees
- moved C3 1.80 mm to (55.9, 123.2), turned to 270 degrees
Connections:
- C2 pad 2: Net-(C2-Pad2) -> GND
- J3 pad 1: Net-(C2-Pad2) -> GND
- T1 pad 5: Net-(C2-Pad2) -> GND
Routing:
- net Net-(C2-Pad1): track 0.00 -> 100.3 mm
- net Net-(C1-Pad1): track 0.23 -> 81.8 mm
- net Net-(C4-Pad1): track 0.00 -> 73.5 mm
- net GND: track 0.00 -> 57.2 mm
- net Net-(D2-Pad2): track 0.00 -> 53.5 mm
- net Net-(C6-Pad2): track 0.00 -> 39.2 mm
- net Net-(D1-Pad2): track 0.00 -> 28.4 mm
- net Net-(Q1-Pad1): track 0.00 -> 23.2 mm
- net Net-(C3-Pad1): track 0.00 -> 22.7 mm
- net Net-(J4-Pad1): track 0.00 -> 16.5 mm
- net Net-(C1-Pad2): track 0.00 -> 15.9 mm
- net Net-(C5-Pad2): track 0.00 -> 6.50 mm
- net Net-(R3-Pad1): track 0.00 -> 6.49 mm
- net Net-(C4-Pad2): track 0.00 -> 4.62 mm
- added copper zone on B.Cu, net GND
- added copper zone on F.Cu, net GND
Other:
- board outline added: 152.4 x 114.3 mm
- board text added: "+15 Vdc"
- board text added: "-15 Vdc"
- board text added: "24-48 Vdc"
- board text added: "Vcc=25V"
