File: PCB_desing/Hardwareproject.sch (KiCad schematic (older format))
At the start: 9 parts, among them J1 Barrel_Jack, Q1 IRF540N, T1 Transformer_1P_1S

Commit message: All PCB is done, average switch network is created and transfer function tested.
Parts:
- removed T1: Transformer_1P_1S, Transformer_THT:Transformer_CHK_EI30-2VA_1xSec, symbol Device:Transformer_1P_1S
- added C3: 18.8nF, Capacitor_THT:C_Disc_D3.4mm_W2.1mm_P2.50mm, symbol Device:CP
- added C4: 470nF, Capacitor_THT:C_Disc_D3.4mm_W2.1mm_P2.50mm, symbol Device:C
- added C5: 100nF, Capacitor_THT:C_Disc_D3.4mm_W2.1mm_P2.50mm, symbol Device:C
- added C6: 10nF, Capacitor_THT:C_Disc_D3.4mm_W2.1mm_P2.50mm, symbol Device:C
- added J2, J3: Conn_01x01, Connector:Banana_Jack_1Pin, symbol Connector_Generic:Conn_01x01
- added J4: Barrel_Jack, Connector_BarrelJack:BarrelJack_CUI_PJ-063AH_Horizontal, symbol Connector:Barrel_Jack
- added R3: 1000, Resistor_THT:R_Axial_DIN0204_L3.6mm_D1.6mm_P5.08mm_Horizontal, symbol Device:R
- added R4: 270 ohm, Resistor_THT:R_Axial_DIN0204_L3.6mm_D1.6mm_P5.08mm_Horizontal, symbol Device:R
- added R5: 30 ohm, Resistor_THT:R_Axial_DIN0204_L3.6mm_D1.6mm_P5.08mm_Horizontal, symbol Device:R
- added R6: 200 ohm, Resistor_THT:R_Axial_DIN0204_L3.6mm_D1.6mm_P5.08mm_Horizontal, symbol Device:R
- added T1: PA0184NL, Transformer_THT:Transformer_CHK_EI54-12VA_1xSec, symbol Transformer:PA0184NL
- added U1: lt1246, Package_DIP:DIP-8_W7.62mm, symbol New_Library_0:lt1246
- C1: value 20u -> 200u; footprint Capacitor_SMD:CP_Elec_4x5.4 -> Capacitor_THT:CP_Radial_D7.5mm_P2.50mm
- C2: value 100u -> 330u; footprint Capacitor_THT:CP_Radial_D7.5mm_P2.50mm -> Capacitor_THT:CP_Radial_D12.5mm_P5.00mm
- D1: value D -> VT3080S; footprint Package_TO_SOT_THT:TO-220-2_Horizontal_TabDown -> Package_TO_SOT_THT:TO-220-2_Vertical
- D2: footprint Package_TO_SOT_THT:TO-220-2_Horizontal_TabDown -> Diode_THT:D_A-405_P7.62mm_Horizontal
- J1: footprint Connector_BarrelJack:BarrelJack_CUI_PJ-102AH_Horizontal -> Connector_BarrelJack:BarrelJack_CUI_PJ-063AH_Horizontal
- R1: value 1k -> 2k; footprint Resistor_SMD:R_0201_0603Metric -> Resistor_THT:R_Axial_DIN0204_L3.6mm_D1.6mm_P5.08mm_Horizontal
- R2: value 3 -> 1k; footprint Resistor_THT:R_Axial_DIN0204_L3.6mm_D1.6mm_P1.90mm_Vertical -> Resistor_THT:R_Axial_DIN0204_L3.6mm_D1.6mm_P5.08mm_Horizontal
Connections:
- net at Q1.1 (G): now also U1.6 (Out)
- net at D2.2 (A), Q1.2 (D): now also T1.8
- net GND: now reaches J1.2, Q1.3 (S)
- net GND: now also C3.2, J4.2, R6.2, U1.3 (Isense), U1.5 (GND)
- net at C1.1, J1.1, R1.1: now also T1.1
- net at C2.2: now also J3.1 (Pin_1), T1.5; no longer R2.2
- net at D1.2 (A): now also T1.4
- net at C2.1, D1.1 (K), R2.1: now also C5.1, J2.1 (Pin_1)
- new net: C6.2, R4.2, U1.1 (Comp)
- new net: C4.1, C6.1, R2.2, R5.2, R6.1, U1.2 (FB)
- new net: C3.1, R3.2, U1.4 (Osc)
- new net: J4.1, U1.7 (Vcc)
- new net: R3.1, U1.8 (Vref)
- new net: C5.2, R5.1
- new net: C4.2, R4.1
- no-connect marks 1 -> 0
Other:
- moved on the sheet: C1, C2, D1, D2, J1, Q1, R1

Commit message: Updates
Parts:
- added HS1, HS2: Heatsink, Heatsink:Heatsink_Stonecold_HS-132_32x14mm_2xFixation1.5mm, symbol Mechanical:Heatsink
- C3, C4, C5, C6: footprint Capacitor_THT:C_Disc_D3.4mm_W2.1mm_P2.50mm -> Capacitor_Tantalum_SMD:CP_EIA-3216-10_Kemet-I
Connections:
- net GND: now also C2.2, J3.1 (Pin_1), T1.5
Other:
- moved on the sheet: C1, C2, C3, C4, C5, C6, D1, D2, J1, J2, J3, J4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
